File: Electronics/commboard/Module_RS485.kicad_sch (KiCad schematic)
At the start: 6 parts, among them J201 RS485_Out_1, U201 SP3485EN

Commit message: completed pcb design
Parts:
- J201: value RS485_Out_1 -> ServoConn; footprint (none) -> Connector_PinHeader_2.54mm:PinHeader_1x04_P2.54mm_Vertical
Connections:
- net 24V_Unsafe renamed ServoPower
Changed lines of the file:
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@@
     (effects (font (size 1.27 1.27)) (justify right))
   )
-  (hierarchical_label "24V_Unsafe" (shape bidirectional) (at 183.642 98.298 0)
+  (hierarchical_label "ServoPower" (shape bidirectional) (at 183.642 98.298 0)
     (effects (font (size 1.27 1.27)) (justify left))
   )
   (symbol (lib_id "Connector:Screw_Terminal_01x04") (at 174.498 84.582 0) (unit 1)
-    (in_bom yes) (on_board yes)
-    (property "Reference" "J201" (id 0) (at 176.784 84.5819 0)
-      (effects (font (size 1.27 1.27)) (justify left))
-    )
-    (property "Value" "RS485_Out_1" (id 1) (at 168.402 92.202 0)
-      (effects (font (size 1.27 1.27)) (justify left))
-    )
-    (property "Footprint" "" (id 2) (at 174.498 84.582 0)
+    (in_bom yes) (on_board yes) (fields_autoplaced)
+    (property "Reference" "J201" (id 0) (at 174.498 93.98 0))
+    (property "Value" "ServoConn" (id 1) (at 174.498 96.52 0))
+    (property "Footprint" "Connector_PinHeader_2.54mm:PinHeader_1x04_P2.54mm_Vertical" (id 2) (at 174.498 84.582 0)
       (effects (font (size 1.27 1.27)) hide)
     )
@@
   (symbol (lib_id "Device:R") (at 146.812 86.614 0) (unit 1)
     (in_bom yes) (on_board yes) (fields_autoplaced)
-    (property "Reference" "R202" (id 0) (at 149.606 85.3439 0)
+    (property "Reference" "R202" (id 0) (at 148.59 85.3439 0)
       (effects (font (size 1.27 1.27)) (justify left))
     )
-    (property "Value" "60R" (id 1) (at 149.606 87.8839 0)
+    (property "Value" "60R" (id 1) (at 148.59 87.8839 0)
       (effects (font (size 1.27 1.27)) (justify left))
     )
@@
   (symbol (lib_id "Device:R") (at 146.812 97.282 0) (unit 1)
     (in_bom yes) (on_board yes) (fields_autoplaced)
-    (property "Reference" "R203" (id 0) (at 149.5239 96.0119 0)
+    (property "Reference" "R203" (id 0) (at 148.59 96.0119 0)
       (effects (font (size 1.27 1.27)) (justify left))
     )
-    (property "Value" "220R" (id 1) (at 149.5239 98.5519 0)
+    (property "Value" "220R" (id 1) (at 148.59 98.5519 0)
       (effects (font (size 1.27 1.27)) (justify left))
     )
@@
   (symbol (lib_id "Interface_UART:SP3485EN") (at 129.54 86.36 0) (unit 1)
     (in_bom yes) (on_board yes) (fields_autoplaced)
-    (property "Reference" "U201" (id 0) (at 131.5594 72.898 0)
+    (property "Reference" "U201" (id 0) (at 131.5594 73.66 0)
       (effects (font (size 1.27 1.27)) (justify left))
     )
-    (property "Value" "SP3485EN" (id 1) (at 131.5594 75.438 0)
+    (property "Value" "SP3485EN" (id 1) (at 131.5594 76.2 0)
       (effects (font (size 1.27 1.27)) (justify left))
     )
@@
   )
   (symbol (lib_id "Device:C") (at 181.864 75.946 0) (unit 1)
-    (in_bom yes) (on_board yes)
-    (property "Reference" "C201" (id 0) (at 175.006 74.676 0)
+    (in_bom yes) (on_board yes) (fields_autoplaced)
+    (property "Reference" "C201" (id 0) (at 185.42 74.6759 0)
       (effects (font (size 1.27 1.27)) (justify left))
     )
-    (property "Value" "100nF" (id 1) (at 173.228 77.47 0)
+    (property "Value" "100nF" (id 1) (at 185.42 77.2159 0)
       (effects (font (size 1.27 1.27)) (justify left))
     )
@@
   (symbol (lib_id "Device:R") (at 146.812 74.93 0) (unit 1)
     (in_bom yes) (on_board yes) (fields_autoplaced)
-    (property "Reference" "R201" (id 0) (at 149.606 73.6599 0)
+    (property "Reference" "R201" (id 0) (at 148.59 73.6599 0)
       (effects (font (size 1.27 1.27)) (justify left))
     )
-    (property "Value" "220R" (id 1) (at 149.606 76.1999 0)
+    (property "Value" "220R" (id 1) (at 148.59 76.1999 0)
       (effects (font (size 1.27 1.27)) (justify left))
     )

Commit message: schematic design completed. pcb layout drawings completed.
Parts:
- J201: footprint Connector_PinHeader_2.54mm:PinHeader_1x04_P2.54mm_Vertical -> Connector_Phoenix_MSTB:PhoenixContact_MSTBVA_2,5_4-G-5,08_1x04_P5.08mm_Vertical
Changed lines of the file:
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@@
   (symbol (lib_id "Connector:Screw_Terminal_01x04") (at 174.498 84.582 0) (unit 1)
     (in_bom yes) (on_board yes) (fields_autoplaced)
-    (property "Reference" "J201" (id 0) (at 174.498 93.98 0))
-    (property "Value" "ServoConn" (id 1) (at 174.498 96.52 0))
-    (property "Footprint" "Connector_PinHeader_2.54mm:PinHeader_1x04_P2.54mm_Vertical" (id 2) (at 174.498 84.582 0)
+    (property "Reference" "J201" (id 0) (at 174.498 74.93 0))
+    (property "Value" "ServoConn" (id 1) (at 174.498 77.47 0))
+    (property "Footprint" "Connector_Phoenix_MSTB:PhoenixContact_MSTBVA_2,5_4-G-5,08_1x04_P5.08mm_Vertical" (id 2) (at 174.498 84.582 0)
       (effects (font (size 1.27 1.27)) hide)
     )
